File: PCB/wififp_receiver/receiver.kicad_pcb (KiCad board)
At the start: 2 copper layers, 17 parts, among them IC1 ATTINY2313-P, P1 ICISP1, P2 USB, U1 rf-receiver, X1 12MHz

Commit message: Updated the schematic
Parts:
- added D1: 1N4148, Diodes_SMD:D_0805, F.Cu at (148.6, 101.6)
- added R7: 1K5, Capacitors_SMD:C_0805_HandSoldering, F.Cu at (146.1, 104.1)
- moved R4 3.81 mm to (149.9, 104.1)
- moved U1 2.54 mm to (151.1, 99.1)
Connections:
- R4 pad 1: Net-(C4-Pad1) -> Net-(D1-Pad2)
Routing:
- net Net-(D1-Pad2): track 0.00 -> 3.95 mm
- net VDD: track 76.7 -> 79.3 mm
- net GNDREF: track 52.0 -> 54.5 mm
